File: pcb/circuit.kicad_pcb (KiCad board)
At the start: 2 copper layers, 32 parts, among them IC1 OP703PA, J1 soldering iron, J2 Conn_01x04_Female, J3 Conn_01x08_Female, Q1 IRF5305, Q2 2N7000, SW1 SW_Push, SW2 SW_Push, SW3 SW_Push, SW4 Rotary_Encoder_Switch, U1 ATmega328-PU, U2 4050

Commit message: v0.0.4
Parts:
- removed A1: Arduino_Nano_v3.x, Module:Arduino_Nano
- removed R11, R12, R13, R15, R16: R, Resistor_THT:R_Axial_DIN0204_L3.6mm_D1.6mm_P7.62mm_Horizontal
- added J4: 12V, Connector_BarrelJack:BarrelJack_CUI_PJ-063AH_Horizontal, F.Cu at (26.7, 52.1)
- added J5: Power 12V, Connector_Phoenix_MSTB:PhoenixContact_MSTBVA_2,5_2-G-5,08_1x02_P5.08mm_Vertical, F.Cu at (19.1, 64.8)
- added J6: LiPo-Bal, Connector_JST:JST_EH_B4B-EH-A_1x04_P2.50mm_Vertical, F.Cu at (19.7, 105.4)
- added J7: Screw_Terminal_01x02, Connector_PinSocket_1.27mm:PinSocket_1x02_P1.27mm_Vertical, F.Cu at (20.3, 146.7)
- added J8: Conn_01x04_Female, Connector_PinHeader_2.54mm:PinHeader_1x04_P2.54mm_Vertical, F.Cu at (27.3, 144.8)
- added J9: ISP, Connector_PinHeader_2.54mm:PinHeader_2x03_P2.54mm_Vertical, F.Cu at (19.1, 86.4)
- added Q3: LM7805, Package_TO_SOT_THT:TO-220-3_Vertical, F.Cu at (34.9, 65.4)
- added Q4: LM117T 3.3, Package_TO_SOT_THT:TO-220-3_Vertical, F.Cu at (35.6, 54.6)
- added R20: 560Ω, Resistor_THT:R_Axial_DIN0204_L3.6mm_D1.6mm_P7.62mm_Horizontal, F.Cu at (130.5, 34.7)
- added R21: 2MΩ, Resistor_THT:R_Axial_DIN0204_L3.6mm_D1.6mm_P7.62mm_Horizontal, F.Cu at (158.0, 19.7)
- added R22: 1MΩ, Resistor_THT:R_Axial_DIN0204_L3.6mm_D1.6mm_P7.62mm_Horizontal, F.Cu at (158.0, 22.9)
- added R23: 1MΩ, Resistor_THT:R_Axial_DIN0204_L3.6mm_D1.6mm_P7.62mm_Horizontal, F.Cu at (156.6, 31.5)
- added R24: 1MΩ, Resistor_THT:R_Axial_DIN0204_L3.6mm_D1.6mm_P7.62mm_Horizontal, F.Cu at (158.0, 26.0)
- added R25: 1MΩ, Resistor_THT:R_Axial_DIN0204_L3.6mm_D1.6mm_P7.62mm_Horizontal, F.Cu at (156.6, 34.7)
- added SW5: T-, Button_Switch_THT:SW_Tactile_Straight_KSL0Axx1LFTR, F.Cu at (268.0, 69.8)
- added SW6: Pow, Button_Switch_THT:SW_Tactile_Straight_KSL0Axx1LFTR, F.Cu at (268.0, 90.2)
- added SW7: Rotary_Encoder_Switch, Rotary_Encoder:RotaryEncoder_Alps_EC11E-Switch_Vertical_H20mm, F.Cu at (25.4, 160.0)
- added U3: LM4040LP-4.1, Package_TO_SOT_THT:TO-92_Inline, F.Cu at (114.9, 44.5)
- added Y1: 16MHz, Crystal:Crystal_HC18-U_Vertical, F.Cu at (169.5, 104.8)
- C1: footprint Capacitor_THT:CP_Axial_L10.0mm_D4.5mm_P15.00mm_Horizontal -> Capacitor_THT:C_Disc_D4.3mm_W1.9mm_P5.00mm
- C2: footprint Capacitor_THT:CP_Radial_D5.0mm_P2.50mm -> Capacitor_THT:C_Disc_D4.3mm_W1.9mm_P5.00mm
- IC1: footprint Package_SO:SOIC-8_3.9x4.9mm_P1.27mm -> Package_DIP:DIP-8_W7.62mm
- J1: value soldering iron -> Soldering iron; footprint Connector_PinHeader_1.27mm:PinHeader_1x04_P1.27mm_Vertical -> Connector_Phoenix_MSTB:PhoenixContact_MSTBVA_2,5_4-G_1x04_P5.00mm_Vertical
- J2: value Conn_01x04_Female -> TFT AK; footprint Connector_PinHeader_1.27mm:PinHeader_1x04_P1.27mm_Vertical -> Connector_PinHeader_2.54mm:PinHeader_1x08_P2.54mm_Vertical
- J3: value Conn_01x08_Female -> TFT RL; footprint Connector_PinHeader_1.27mm:PinHeader_1x08_P1.27mm_Horizontal -> Connector_PinHeader_2.54mm:PinHeader_1x08_P2.54mm_Vertical
- SW1: value SW_Push -> T1
- SW2: value SW_Push -> T2
- SW3: value SW_Push -> T3
- SW4: value Rotary_Encoder_Switch -> T+; footprint Rotary_Encoder:RotaryEncoder_Alps_EC11E-Switch_Vertical_H20mm -> Button_Switch_THT:SW_Tactile_Straight_KSL0Axx1LFTR
- moved J1 246.5 mm to (20.3, 20.3), turned to 270 degrees
- moved R10 193.0 mm to (271.8, 133.3), turned to 180 degrees
- moved Q1 190.5 mm to (35.6, 20.3), turned to 0 degrees
- moved Q2 183.0 mm to (35.6, 35.6), turned to 90 degrees
- moved SW4 166.2 mm to (268.0, 50.8)
- moved D1 141.3 mm to (267.3, 122.6)
- moved J3 134.5 mm to (232.4, 38.1)
- moved J2 125.0 mm to (240.0, 38.1)
- moved U2 123.1 mm to (212.7, 38.1)
- moved SW3 113.3 mm to (224.8, 121.9)
- moved U1 109.6 mm to (144.8, 94.0), turned to 90 degrees
- moved SW2 103.9 mm to (208.3, 121.9)
- moved SW1 97.3 mm to (191.8, 121.9)
- moved R14 91.8 mm to (96.5, 15.9), turned to 0 degrees
- moved IC1 78.0 mm to (96.5, 48.3)
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Connections:
- C2 pad 1: Net-(C2-Pad1) -> GNDD
- C2 pad 2: Net-(C2-Pad2) -> Sensor
- D1 pad 1: Net-(D1-Pad1) -> GNDD
- J2 pad 2: Net-(J2-Pad2) -> GNDD
- J3 pad 1: Net-(J3-Pad1) -> GNDD
- J3 pad 2: Net-(J3-Pad2) -> +3V3
- J3 pad 3: Net-(J3-Pad3) -> Net-(J2-Pad5)
- J3 pad 4: Net-(J3-Pad4) -> Net-(J2-Pad4)
- J3 pad 5: Net-(J3-Pad5) -> Net-(J2-Pad1)
- J3 pad 6: Net-(J3-Pad6) -> Net-(J2-Pad3)
- J3 pad 7: Net-(J3-Pad7) -> GNDD
- J3 pad 8: Net-(J3-Pad8) -> +3V3
- R10 pad 1: Net-(R10-Pad1) -> Net-(D1-Pad2)
- R5 pad 1: Net-(A1-Pad19) -> Sensor
- R8 pad 1: Net-(A1-Pad6) -> Tip
- SW1 pad 1: Net-(SW1-Pad1) -> GNDD
- SW1 pad 2: Net-(SW1-Pad2) -> T1
- SW2 pad 1: Net-(SW2-Pad1) -> GNDD
- SW2 pad 2: Net-(SW2-Pad2) -> T2
- SW3 pad 1: Net-(SW3-Pad1) -> GNDD
- SW3 pad 2: Net-(SW3-Pad2) -> T3
- U1 pad 1: Net-(U1-Pad1) -> Res
- U1 pad 11: Net-(U1-Pad11) -> T-
- U1 pad 12: Net-(U1-Pad12) -> Pow
- U1 pad 13: Net-(U1-Pad13) -> Net-(R10-Pad2)
- U1 pad 15: Net-(U1-Pad15) -> DC
- U1 pad 16: Net-(U1-Pad16) -> CS
- U1 pad 17: Net-(U1-Pad17) -> SDA
- U1 pad 18: Net-(U1-Pad18) -> MISO
- U1 pad 19: Net-(U1-Pad19) -> SCL
- U1 pad 2: Net-(U1-Pad2) -> T1
- U1 pad 21: Net-(U1-Pad21) -> +12C
- U1 pad 23: Net-(U1-Pad23) -> Sensor
- U1 pad 24: Net-(U1-Pad24) -> LiPo3
- U1 pad 25: Net-(U1-Pad25) -> LiPo2
- U1 pad 26: Net-(U1-Pad26) -> LiPo1
- U1 pad 3: Net-(U1-Pad3) -> T2
- U1 pad 4: Net-(U1-Pad4) -> T3
- U1 pad 5: Net-(U1-Pad5) -> Tip
- U1 pad 6: Net-(U1-Pad6) -> T+
- U2 pad 1: Net-(U2-Pad1) -> +3V3
- U2 pad 10: Net-(U2-Pad10) -> Net-(J2-Pad4)
- U2 pad 11: Net-(U2-Pad11) -> SCL
- U2 pad 12: Net-(U2-Pad12) -> Net-(J2-Pad5)
- U2 pad 2: Net-(U2-Pad2) -> GNDD
- U2 pad 3: Net-(U2-Pad3) -> CS
- U2 pad 4: Net-(U2-Pad4) -> Net-(J2-Pad3)
- U2 pad 5: Net-(U2-Pad5) -> DC
- U2 pad 6: Net-(U2-Pad6) -> Net-(J2-Pad1)
- U2 pad 7: Net-(U2-Pad7) -> Res
- U2 pad 8: Net-(U2-Pad8) -> GNDD
- U2 pad 9: Net-(U2-Pad9) -> SDA
Routing:
- net T-: track 0.00 -> 117.4 mm
- net Net-(Q1-Pad1): track 94.0 -> 0.00 mm
- net GNDD: track 0.00 -> 92.2 mm
- net Pow: track 0.00 -> 84.8 mm
- net +12C: track 43.2 -> 0.00 mm
- net Net-(J1-Pad1): track 42.2 -> 0.00 mm
- net Net-(D1-Pad2): track 0.00 -> 11.6 mm
Other:
- net class Neu added: clearance 0.5, trace_width 0.25, via_dia 0.8, via_drill 0.4

Commit message: v0.0.7
Parts:
- removed SW4: T+, Button_Switch_THT:SW_Tactile_Straight_KSL0Axx1LFTR
- removed SW5: T-, Button_Switch_THT:SW_Tactile_Straight_KSL0Axx1LFTR
- removed SW6: Pow, Button_Switch_THT:SW_Tactile_Straight_KSL0Axx1LFTR
- added A1: Arduino_Nano_v3.x, Module:Arduino_Nano, F.Cu at (110.3, 42.2)
- added JP1: USE_TFT_RESET, Connector_PinHeader_2.54mm:PinHeader_1x03_P2.54mm_Vertical, F.Cu at (204.8, 162.4)
- added JP2: Backlight, Connector_PinHeader_2.54mm:PinHeader_1x03_P2.54mm_Vertical, F.Cu at (80.5, 59.2)
- added Q5: BC328, Package_TO_SOT_THT:TO-92_Inline, F.Cu at (147.5, 112.2)
- added R20: 560Ω, Resistor_THT:R_Axial_DIN0204_L3.6mm_D1.6mm_P7.62mm_Horizontal, F.Cu at (31.7, 69.9)
- added TR1: Backlight, Potentiometer_THT:Potentiometer_Piher_PT-10-V10_Vertical, F.Cu at (270.1, 102.4)
- added U4: TXS0102DCT, Package_SO:SSOP-8_2.95x2.8mm_P0.65mm, F.Cu at (66.2, 117.4)
- J2: footprint Connector_PinHeader_2.54mm:PinHeader_1x08_P2.54mm_Vertical -> my:TFT-1.8-AK
- J3: footprint Connector_PinHeader_2.54mm:PinHeader_1x08_P2.54mm_Vertical -> my:TFT-1.8-RGB
- J8: value Conn_01x04_Female -> I2C
- R11: renamed from R20; value 560Ω -> R
- SW7: value Rotary_Encoder_Switch -> Menu
- moved SW7 270.3 mm to (275.8, 58.3), turned to 270 degrees
- moved R5 230.0 mm to (315.5, 34.2)
- moved R8 224.1 mm to (282.5, 31.6), turned to 90 degrees
- moved Q4 222.0 mm to (255.5, 24.0), turned to 270 degrees
- moved Q3 202.0 mm to (232.7, 24.1), turned to 270 degrees
- moved R7 193.2 mm to (279.2, 24.0), turned to 270 degrees
- moved R11 177.7 mm to (305.3, 67.1)
- moved J4 175.0 mm to (201.2, 64.8)
- moved Q1 174.9 mm to (210.5, 24.1), turned to 270 degrees
- moved J5 174.6 mm to (192.9, 48.8)
- moved J1 172.6 mm to (192.8, 25.2)
- moved J6 172.5 mm to (190.6, 82.3), turned to 90 degrees
- moved Q2 165.8 mm to (201.0, 23.8), turned to 0 degrees
- moved C1 163.4 mm to (230.6, 47.1), turned to 0 degrees
- moved R6 159.6 mm to (206.5, 31.5), turned to 90 degrees
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Connections:
- IC1 pad 7: +12C -> +5V
- J2 pad 2: GNDD -> Net-(J2-Pad2)
- J2 pad 7: +3V3 -> Net-(J2-Pad7)
- J3 pad 7: GNDD -> Net-(J2-Pad2)
- J3 pad 8: +3V3 -> Net-(J2-Pad7)
- J8 pad 1: Net-(J8-Pad1) -> +5V
- J8 pad 4: Net-(J8-Pad4) -> GNDD
- J9 pad 3: SCL -> SCK
- J9 pad 4: SDA -> MOSI
- R11 pad 1: +12C -> Net-(Q5-Pad2)
- R11 pad 2: Net-(R20-Pad2) -> Net-(JP2-Pad2)
- R14 pad 1: +12C -> +5V
- SW3 pad 2: T3 -> MISO
- SW7 pad A: Net-(SW7-PadA) -> T-
- SW7 pad B: Net-(SW7-PadB) -> T+
- SW7 pad C: Net-(SW7-PadC) -> GNDD
- SW7 pad S1: Net-(SW7-PadS1) -> Pow
- SW7 pad S2: Net-(SW7-PadS2) -> GNDD
- U1 pad 12: Pow -> BL
- U1 pad 14: Net-(U1-Pad14) -> TFT-RST
- U1 pad 17: SDA -> MOSI
- U1 pad 19: SCL -> SCK
- U1 pad 27: Net-(U1-Pad27) -> SDA
- U1 pad 28: Net-(U1-Pad28) -> SCL
- U1 pad 4: T3 -> Pow
- U2 pad 11: SCL -> SCK
- U2 pad 14: (no net) -> Net-(U2-Pad14)
- U2 pad 15: (no net) -> Net-(U2-Pad15)
- U2 pad 2: GNDD -> Net-(J2-Pad2)
- U2 pad 7: Res -> Net-(JP1-Pad2)
- U2 pad 9: SDA -> MOSI
Routing:
- net +12C: track 0.00 -> 157.7 mm
- net T-: track 117.4 -> 0.00 mm
- net Pow: track 84.8 -> 0.00 mm
- net Net-(Q2-Pad2): track 0.00 -> 83.0 mm
- net GNDD: track 92.2 -> 174.0 mm
- net Net-(J1-Pad2): track 0.00 -> 19.9 mm
- net Net-(J1-Pad1): track 0.00 -> 18.2 mm
- net Net-(D1-Pad2): track 11.6 -> 0.00 mm
- net Net-(Q1-Pad1): track 0.00 -> 7.04 mm
- net Net-(J6-Pad3): track 0.00 -> 5.14 mm
- net Net-(J6-Pad2): track 0.00 -> 5.12 mm
- net Net-(J6-Pad1): track 0.00 -> 5.12 mm
- added copper zone on F.Cu, net (none)

Commit message: v0.0.8
Parts:
- removed J7: Screw_Terminal_01x02, Connector_PinSocket_1.27mm:PinSocket_1x02_P1.27mm_Vertical
- removed R9: R, Resistor_THT:R_Axial_DIN0204_L3.6mm_D1.6mm_P7.62mm_Horizontal
- moved Y1 203.3 mm to (247.5, 93.4), turned to 180 degrees
- moved C2 194.1 mm to (246.8, 48.4)
- moved JP2 183.1 mm to (259.1, 99.3), turned to 90 degrees
- moved R20 172.0 mm to (202.2, 47.2)
- moved R4 171.0 mm to (244.5, 43.4), turned to 90 degrees
- moved R3 163.6 mm to (236.5, 51.1), turned to 180 degrees
- moved R24 153.9 mm to (229.7, 75.6)
- moved Q5 151.0 mm to (280.8, 41.1)
- moved U3 138.8 mm to (214.9, 47.2)
- moved R25 138.5 mm to (203.4, 85.1), turned to 180 degrees
- moved U4 133.6 mm to (198.8, 101.6), turned to 270 degrees
- moved J8 132.3 mm to (190.8, 106.0), turned to 180 degrees
- moved U2 97.1 mm to (226.2, 66.9)
- moved R10 89.0 mm to (265.9, 86.9)
- moved D1 87.3 mm to (270.9, 58.6), turned to 270 degrees
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Connections:
- U1 pad 21: +12C -> VMEM
- U1 pad 22: Net-(U1-Pad22) -> GNDD
- U1 pad 7: Net-(U1-Pad7) -> +5V
- U1 pad 8: Net-(U1-Pad22) -> GNDD
- U2 pad 14: Net-(U2-Pad14) -> (no net)
- U2 pad 15: Net-(U2-Pad15) -> (no net)
Routing:
- net GNDD: track 174.0 -> 259.4 mm
- net BL: track 0.00 -> 14.2 mm
- net +12C: track 157.7 -> 152.0 mm
- added copper zone on B.Cu, net (none)
Other:
- net class Default: clearance 0.2 -> 0.3
- net class Neu removed
- net class Original added: clearance 0.2, trace_width 0.25, via_dia 0.8, via_drill 0.4
- rule trace_clearance: 0.2 -> 0.3
- rule trace_min: 0.2 -> 0.5

Commit message: v0.0.10
Parts:
- removed JP2: Backlight, Connector_PinHeader_2.54mm:PinHeader_1x03_P2.54mm_Vertical
- removed Q5: BC328, Package_TO_SOT_THT:TO-92_Inline
- removed R11: R, Resistor_THT:R_Axial_DIN0204_L3.6mm_D1.6mm_P7.62mm_Horizontal
- removed TR1: Backlight, Potentiometer_THT:Potentiometer_Piher_PT-10-V10_Vertical
- U4: footprint Package_SO:SSOP-8_2.95x2.8mm_P0.65mm -> Package_DIP:DIP-8_W7.62mm
- moved U4 13.1 mm to (210.1, 108.4)
- moved J2 3.64 mm to (208.1, 51.5)
- moved C2 2.71 mm to (248.2, 46.1)
- moved R3 1.65 mm to (236.4, 49.4)
Connections:
- J2 pad 6: +3V3 -> Net-(J2-Pad6)
- J3 pad 2: +3V3 -> Net-(J2-Pad6)
- U2 pad 1: +3V3 -> Net-(J2-Pad6)
- U2 pad 14: (no net) -> BL
- U2 pad 15: (no net) -> Net-(J2-Pad7)
Routing:
- removed copper zone on B.Cu, net (none)

Commit message: v0.0.11
Parts:
- added C3: 100nF, Capacitor_THT:C_Disc_D4.3mm_W1.9mm_P5.00mm, F.Cu at (105.7, 121.2)
- added C4: 100nF, Capacitor_THT:C_Disc_D4.3mm_W1.9mm_P5.00mm, F.Cu at (102.3, 130.9)
- added C5: 100nF, Capacitor_THT:C_Disc_D4.3mm_W1.9mm_P5.00mm, F.Cu at (105.7, 124.6)
- added JP2: BL Control, Connector_PinHeader_2.54mm:PinHeader_1x03_P2.54mm_Vertical, F.Cu at (101.8, 121.8)
- added R9: 10kΩ, Resistor_THT:R_Axial_DIN0204_L3.6mm_D1.6mm_P7.62mm_Horizontal, F.Cu at (91.6, 133.3)
- J1: footprint Connector_Phoenix_MSTB:PhoenixContact_MSTBVA_2,5_4-G_1x04_P5.00mm_Vertical -> TerminalBlock_Phoenix:TerminalBlock_Phoenix_MKDS-1,5-4-5.08_1x04_P5.08mm_Horizontal
- J5: footprint Connector_Phoenix_MSTB:PhoenixContact_MSTBVA_2,5_2-G-5,08_1x02_P5.08mm_Vertical -> TerminalBlock_Phoenix:TerminalBlock_Phoenix_MKDS-1,5-2-5.08_1x02_P5.08mm_Horizontal
- JP1: value USE_TFT_RESET -> TFT Reset
- Q1, Q3, Q4: footprint Package_TO_SOT_THT:TO-220-3_Vertical -> Package_TO_SOT_THT:TO-220-3_Horizontal_TabDown
- Y1: footprint Crystal:Crystal_HC18-U_Vertical -> Crystal:Crystal_HC49-U_Vertical
- moved C2 209.6 mm to (40.6, 75.2), turned to 90 degrees
- moved R5 201.2 mm to (40.6, 67.6)
- moved R4 194.0 mm to (51.2, 59.9), turned to 180 degrees
- moved R3 184.9 mm to (51.6, 49.4), turned to 270 degrees
- moved C1 181.3 mm to (50.3, 47.0)
- moved U3 180.5 mm to (34.5, 39.5), turned to 270 degrees
- moved IC1 178.0 mm to (48.5, 49.5), turned to 270 degrees
- moved U4 170.8 mm to (39.4, 101.6)
- moved J4 167.2 mm to (34.0, 65.8)
- moved J5 166.5 mm to (26.5, 51.0)
- moved J1 166.4 mm to (26.5, 29.5)
- moved R7 166.1 mm to (113.0, 22.4)
- moved R8 166.0 mm to (117.0, 45.5)
- moved R14 165.2 mm to (46.1, 37.3), turned to 180 degrees
- moved D1 164.9 mm to (106.4, 70.0)
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Connections:
- net T+ renamed Up
- net T- renamed Down
- J2 pad 6: Net-(J2-Pad6) -> +5V
- J3 pad 2: Net-(J2-Pad6) -> +5V
- J4 pad 1: +12C -> +12V
- J5 pad 1: +12C -> +12V
- Q1 pad 3: +12C -> +12V
- Q3 pad 1: +12C -> +12V
- Q4 pad 1: +12C -> +12V
- R20 pad 1: +12C -> AREF
- R20 pad 2: Net-(R20-Pad2) -> +5V
- R6 pad 1: +12C -> +12V
- U1 pad 20: Net-(U1-Pad20) -> +5V
- U1 pad 21: VMEM -> AREF
- U2 pad 1: Net-(J2-Pad6) -> +5V
- U2 pad 14: BL -> Net-(JP2-Pad2)
- U3 pad 2: Net-(R20-Pad2) -> AREF
Routing:
- net +12C: track 152.0 -> 0.00 mm
- net +12V: track 0.00 -> 88.2 mm
- net GNDD: track 259.4 -> 229.3 mm
- net Net-(C1-Pad1): track 0.00 -> 17.0 mm
- net Net-(Q2-Pad2): track 83.0 -> 75.5 mm
- net +5V: track 0.00 -> 6.20 mm
- net AREF: track 0.00 -> 4.57 mm
- net Net-(J1-Pad2): track 19.9 -> 15.5 mm
- net Net-(J1-Pad1): track 18.2 -> 20.2 mm
- removed copper zone on F.Cu, net (none)
Other:
- board outline added: 100 x 100 mm
