File: pcb/circuit.sch (KiCad schematic (older format))
At the start: 37 parts, among them IC1 OP703PA, J1 soldering iron, Q1 IRF5305, Q2 2N7000

Commit message: v0.0.2
Parts:
- C1: footprint (none) -> Capacitor_THT:CP_Axial_L10.0mm_D4.5mm_P15.00mm_Horizontal
- C2: renamed from C?; footprint (none) -> Capacitor_THT:CP_Radial_D5.0mm_P2.50mm
- D1: renamed from D?; footprint (none) -> Diode_THT:D_DO-15_P2.54mm_Vertical_AnodeUp
- J1: footprint (none) -> Connector_PinHeader_1.27mm:PinHeader_1x04_P1.27mm_Vertical
- J2: renamed from J?; footprint (none) -> Connector_PinHeader_1.27mm:PinHeader_1x04_P1.27mm_Vertical
- J3: renamed from J?; footprint (none) -> Connector_PinHeader_1.27mm:PinHeader_1x08_P1.27mm_Horizontal
- R1, R14, R2, R3, R4, R5, R6, R7, R8: footprint (none) -> Resistor_THT:R_Axial_DIN0204_L3.6mm_D1.6mm_P7.62mm_Horizontal
- R10, R11, R12, R13, R15, R16, R9: renamed from R?; footprint (none) -> Resistor_THT:R_Axial_DIN0204_L3.6mm_D1.6mm_P7.62mm_Horizontal
- SW1, SW2, SW3: renamed from SW?; footprint (none) -> Button_Switch_THT:SW_Tactile_Straight_KSL0Axx1LFTR
- SW4: renamed from SW?; footprint (none) -> Rotary_Encoder:RotaryEncoder_Alps_EC11E-Switch_Vertical_H20mm
- U2: renamed from U?; footprint (none) -> Package_DIP:DIP-16_W7.62mm
- gave numbers to parts that had none: 2
Connections:
- wire segments 37 -> 44

Commit message: v0.0.4
Parts:
- removed A1: Arduino_Nano_v3.x, Module:Arduino_Nano, symbol MCU_Module:Arduino_Nano_v3.x
- removed J1: soldering iron, Connector_PinHeader_1.27mm:PinHeader_1x04_P1.27mm_Vertical, symbol Connector:Conn_01x04_Female
- removed J3: Conn_01x08_Female, Connector_PinHeader_1.27mm:PinHeader_1x08_P1.27mm_Horizontal, symbol Connector:Conn_01x08_Female
- removed R12, R13, R15, R16: R, Resistor_THT:R_Axial_DIN0204_L3.6mm_D1.6mm_P7.62mm_Horizontal, symbol Device:R
- added J1: Soldering iron, Connector_Phoenix_MSTB:PhoenixContact_MSTBVA_2,5_4-G_1x04_P5.00mm_Vertical, symbol Connector:Screw_Terminal_01x04
- added J2: TFT AK, Connector_PinHeader_2.54mm:PinHeader_1x08_P2.54mm_Vertical, symbol Connector:Conn_01x08_Male
- added J3: TFT RL, Connector_PinHeader_2.54mm:PinHeader_1x08_P2.54mm_Vertical, symbol Connector:Conn_01x08_Male
- added J4: 12V, Connector_BarrelJack:BarrelJack_CUI_PJ-063AH_Horizontal, symbol Connector:Barrel_Jack
- added J5: Power 12V, Connector_Phoenix_MSTB:PhoenixContact_MSTBVA_2,5_2-G-5,08_1x02_P5.08mm_Vertical, symbol Connector:Screw_Terminal_01x02
- added J6: LiPo-Bal, Connector_JST:JST_EH_B4B-EH-A_1x04_P2.50mm_Vertical, symbol Connector:Conn_01x04_Female
- added J7: Screw_Terminal_01x02, Connector_PinSocket_1.27mm:PinSocket_1x02_P1.27mm_Vertical, symbol Connector:Screw_Terminal_01x02
- added J9: ISP, Connector_PinHeader_2.54mm:PinHeader_2x03_P2.54mm_Vertical, symbol Connector_Generic:Conn_02x03_Odd_Even
- added Q3: LM7805, Package_TO_SOT_THT:TO-220-3_Vertical, symbol Regulator_Linear:LM7805_TO220
- added Q4: LM117T 3.3, Package_TO_SOT_THT:TO-220-3_Vertical, symbol Regulator_Linear:LM7805_TO220
- added R21: 2MΩ, Resistor_THT:R_Axial_DIN0204_L3.6mm_D1.6mm_P7.62mm_Horizontal, symbol Device:R
- added R22, R23, R24, R25: 1MΩ, Resistor_THT:R_Axial_DIN0204_L3.6mm_D1.6mm_P7.62mm_Horizontal, symbol Device:R
- added SW1: T1, Button_Switch_THT:SW_Tactile_Straight_KSL0Axx1LFTR, symbol Switch:SW_Push
- added SW2: T2, Button_Switch_THT:SW_Tactile_Straight_KSL0Axx1LFTR, symbol Switch:SW_Push
- added SW3: T3, Button_Switch_THT:SW_Tactile_Straight_KSL0Axx1LFTR, symbol Switch:SW_Push
- added U3: LM4040LP-4.1, Package_TO_SOT_THT:TO-92_Inline, symbol Reference_Voltage:LM4040LP-4.1
- added Y1: 16MHz, Crystal:Crystal_HC18-U_Vertical, symbol Device:Crystal
- C1: footprint Capacitor_THT:CP_Axial_L10.0mm_D4.5mm_P15.00mm_Horizontal -> Capacitor_THT:C_Disc_D4.3mm_W1.9mm_P5.00mm
- C2: footprint Capacitor_THT:CP_Radial_D5.0mm_P2.50mm -> Capacitor_THT:C_Disc_D4.3mm_W1.9mm_P5.00mm
- IC1: footprint Package_SO:SOIC-8_3.9x4.9mm_P1.27mm -> Package_DIP:DIP-8_W7.62mm
- J8: renamed from J2; footprint Connector_PinHeader_1.27mm:PinHeader_1x04_P1.27mm_Vertical -> Connector_PinHeader_2.54mm:PinHeader_1x04_P2.54mm_Vertical
- R20: renamed from R11; value R -> 560Ω
- SW4: renamed from SW1; value SW_Push -> T+
- SW5: renamed from SW2; value SW_Push -> T-
- SW6: renamed from SW3; value SW_Push -> Pow
- renumbered SW4 to SW7
Connections:
- net labels added: +3.3V, +3V3, +5V, CS, DC, LiPo1, LiPo2, LiPo3, MISO, Pow, Res, SCL, SDA, Sensor, T+, T-, T1, T2, T3, Tip, VMEM
- wire segments 44 -> 114
Other:
- note added: "J1:\n1=Tip\n2=Sensor\n3=Switch/LED\n4 Gnd"
- note added: "Ohne LiPo:\nR21/R22 entfallen\nR23, R24, R25=10kΩ\nPin 3-4 gebrückt"
- note removed: "J1: 1=Tip, 2=Sensor, 3=Switch/LED, 4 Gnd"

Commit message: v0.0.7
Parts:
- added A1: Arduino_Nano_v3.x, Module:Arduino_Nano, symbol MCU_Module:Arduino_Nano_v3.x
- added JP1: USE_TFT_RESET, Connector_PinHeader_2.54mm:PinHeader_1x03_P2.54mm_Vertical, symbol Device:Jumper_NC_Dual
- added JP2: Backlight, Connector_PinHeader_2.54mm:PinHeader_1x03_P2.54mm_Vertical, symbol Jumper:Jumper_3_Open
- added Q5: BC328, Package_TO_SOT_THT:TO-92_Inline, symbol Transistor_BJT:BC328
- added R11: R, Resistor_THT:R_Axial_DIN0204_L3.6mm_D1.6mm_P7.62mm_Horizontal, symbol Device:R
- added TR1: Backlight, Potentiometer_THT:Potentiometer_Piher_PT-10-V10_Vertical, symbol Device:R_POT_TRIM
- added unit 6 of U2
- added U4: TXS0102DCT, Package_SO:SSOP-8_2.95x2.8mm_P0.65mm, symbol Logic_LevelTranslator:TXS0102DCT
- J2: footprint Connector_PinHeader_2.54mm:PinHeader_1x08_P2.54mm_Vertical -> my:TFT-1.8-AK
- J3: footprint Connector_PinHeader_2.54mm:PinHeader_1x08_P2.54mm_Vertical -> my:TFT-1.8-RGB
- J8: value Conn_01x04_Female -> I2C
- SW7: value Rotary_Encoder_Switch -> Menu
Connections:
- net +12C: no longer IC1.7 (V+), R14.1
- net +3V3: now also Q5.1 (C), TR1.1, U4.7 (VCCB); no longer J2.7 (Pin_7), J3.8 (Pin_8)
- net +5V: now also IC1.7 (V+), J8.1 (Pin_1), R14.1, U4.3 (VCCA), U4.6 (OE)
- net GNDD: now also J8.4 (Pin_4), SW7.C, SW7.S2, TR1.3, U4.2 (GND); no longer J2.2 (Pin_2), J3.7 (Pin_7), SW4.1, SW5.1, SW6.1, U2.2
- net MISO: now also SW3.2
- net Pow: now also SW7.S1, U1.4 (PD2); no longer SW6.2, U1.12 (PD6)
- net Res: now also JP1.1; no longer U2.7
- net SCL: now also U1.28 (PC5), U4.1 (B2); no longer J9.3 (Pin_3), U1.19 (PB5), U2.11
- net SDA: now also U1.27 (PC4), U4.8 (B1); no longer J9.4 (Pin_4), U1.17 (PB3), U2.9
- net T+: now also SW7.B; no longer SW4.2
- net T-: now also SW7.A; no longer SW5.2
- net T3: no longer SW3.2, U1.4 (PD2)
- net TFT-RST: now reaches U1.14 (PB0)
- net TFT-RST: now also JP1.3
- net at J8.2 (Pin_2): now also U4.5 (A1)
- net at J8.3 (Pin_3): now also U4.4 (A2)
- new net: J2.2 (Pin_2), J3.7 (Pin_7), U2.2
- new net: JP1.2, U2.7
- new net: Q5.2 (B), R11.1
- new net: J2.7 (Pin_7), J3.8 (Pin_8), Q5.3 (E)
- new net: JP2.2 (C), R11.2
- new net: JP2.3 (B), TR1.2
- new net BL: JP2.1 (A), U1.12 (PD6)
- new net MOSI: J9.4 (Pin_4), U1.17 (PB3), U2.9
- new net SCK: J9.3 (Pin_3), U1.19 (PB5), U2.11

Commit message: v0.0.8
Parts:
- removed J7: Screw_Terminal_01x02, Connector_PinSocket_1.27mm:PinSocket_1x02_P1.27mm_Vertical, symbol Connector:Screw_Terminal_01x02
- removed R9: R, Resistor_THT:R_Axial_DIN0204_L3.6mm_D1.6mm_P7.62mm_Horizontal, symbol Device:R
- removed SW4: T+, Button_Switch_THT:SW_Tactile_Straight_KSL0Axx1LFTR, symbol Switch:SW_Push
- removed SW5: T-, Button_Switch_THT:SW_Tactile_Straight_KSL0Axx1LFTR, symbol Switch:SW_Push
- removed SW6: Pow, Button_Switch_THT:SW_Tactile_Straight_KSL0Axx1LFTR, symbol Switch:SW_Push
- removed unit 6 of U2
Connections:
- net +12C: no longer U1.21 (AREF)
- net +5V: now also U1.7 (VCC)
- net GNDD: now also U1.22 (GND), U1.8 (GND)
- new net VMEM: U1.21 (AREF)
Changed lines of the file:
@@
-$EndComp
-$Comp
-L Switch:SW_Push SW4
-U 1 1 5E4FBC7D
-P 900 6950
-F 0 "SW4" H 900 7235 50  0000 C CNN
-F 1 "T+" H 900 7144 50  0000 C CNN
-F 2 "Button_Switch_THT:SW_Tactile_Straight_KSL0Axx1LFTR" H 900 7150 50  0001 C CNN
-F 3 "~" H 900 7150 50  0001 C CNN
-	1    900  6950
-	1    0    0    -1
-$EndComp
-$Comp
-L Switch:SW_Push SW5
-U 1 1 5E4FD724
-P 900 7300
-F 0 "SW5" H 900 7585 50  0000 C CNN
-F 1 "T-" H 900 7494 50  0000 C CNN
-F 2 "Button_Switch_THT:SW_Tactile_Straight_KSL0Axx1LFTR" H 900 7500 50  0001 C CNN
-F 3 "~" H 900 7500 50  0001 C CNN
-	1    900  7300
-	1    0    0    -1
-$EndComp
-$Comp
-L Switch:SW_Push SW6
-U 1 1 5E4FEE8B
-P 900 7700
-F 0 "SW6" H 900 7985 50  0000 C CNN
-F 1 "Pow" H 900 7894 50  0000 C CNN
-F 2 "Button_Switch_THT:SW_Tactile_Straight_KSL0Axx1LFTR" H 900 7900 50  0001 C CNN
-F 3 "~" H 900 7900 50  0001 C CNN
-	1    900  7700
-	1    0    0    -1
 $EndComp
 $Comp
@@
 $EndComp
 $Comp
-L Device:R R9
-U 1 1 5E50773B
-P 2250 7150
-F 0 "R9" H 2320 7196 50  0000 L CNN
-F 1 "R" H 2320 7105 50  0000 L CNN
-F 2 "Resistor_THT:R_Axial_DIN0204_L3.6mm_D1.6mm_P7.62mm_Horizontal" V 2180 7150 50  0001 C CNN
-F 3 "~" H 2250 7150 50  0001 C CNN
-	1    2250 7150
-	1    0    0    -1
-$EndComp
-$Comp
 L Device:R R10
 U 1 1 5E5093D0
@@
 Wire Wire Line
 	9750 2450 9600 2450
-$Comp
-L Connector:Screw_Terminal_01x02 J7
-U 1 1 5E6EF2BD
-P 1700 7550
-F 0 "J7" H 1780 7542 50  0000 L CNN
-F 1 "Screw_Terminal_01x02" H 1780 7451 50  0000 L CNN
-F 2 "Connector_PinSocket_1.27mm:PinSocket_1x02_P1.27mm_Vertical" H 1700 7550 50  0001 C CNN
-F 3 "~" H 1700 7550 50  0001 C CNN
-	1    1700 7550
-	1    0    0    -1
-$EndComp
 Text GLabel 6500 2450 2    50   Input ~ 0
 LiPo1
@@
 $EndComp
 Wire Wire Line
-	1400 1000 1650 1000
-Wire Wire Line
 	1650 1000 1650 1200
 Wire Wire Line
@@
 	0    1    -1   0
 $EndComp
-Connection ~ 1650 1000
-Wire Wire Line
-	1650 1000 2000 1000
 Connection ~ 7600 1550
 Wire Wire Line
@@
 	1    0    0    -1
 $EndComp
-$Comp
-L 4xxx:4050 U2
-U 6 1 5E58DBB8
-P 1650 7200
-F 0 "U2" H 1650 7517 50  0000 C CNN
-F 1 "4050" H 1650 7426 50  0000 C CNN
-F 2 "Package_DIP:DIP-16_W7.62mm" H 1650 7200 50  0001 C CNN
-F 3 "http://www.intersil.com/content/dam/intersil/documents/cd40/cd4050bms.pdf" H 1650 7200 50  0001 C CNN
-	6    1650 7200
-	1    0    0    -1
-$EndComp
 Wire Wire Line
 	8600 4750 8800 4750
@@
 	8100 2850 8100 2900
 $Comp
+L Logic_LevelTranslator:TXS0102DCT U4
+U 1 1 5E6CF7FC
+P 1700 4600
+F 0 "U4" H 1700 4011 50  0000 C CNN
+F 1 "TXS0102DCT" H 1700 3920 50  0000 C CNN
+F 2 "Package_SO:SSOP-8_2.95x2.8mm_P0.65mm" H 1700 4050 50  0001 C CNN
+F 3 "http://www.ti.com/lit/gpn/txs0102" H 1700 4580 50  0001 C CNN
+	1    1700 4600
+	1    0    0    -1
+$EndComp
+$Comp
+L power:GNDD #PWR0121
+U 1 1 5E7470E9
+P 1700 5100
+F 0 "#PWR0121" H 1700 4850 50  0001 C CNN
+F 1 "GNDD" H 1704 4945 50  0000 C CNN
+F 2 "" H 1700 5100 50  0001 C CNN
+F 3 "" H 1700 5100 50  0001 C CNN
+	1    1700 5100
+	1    0    0    -1
+$EndComp
+$Comp
+L power:+5V #PWR0122
+U 1 1 5E74AF37
+P 1600 4100
+F 0 "#PWR0122" H 1600 3950 50  0001 C CNN
+F 1 "+5V" H 1615 4273 50  0000 C CNN
+F 2 "" H 1600 4100 50  0001 C CNN
+F 3 "" H 1600 4100 50  0001 C CNN
+	1    1600 4100
+	1    0    0    -1
+$EndComp
+$Comp
+L power:+3.3V #PWR0123
+U 1 1 5E74C9C1
+P 1800 4100
+F 0 "#PWR0123" H 1800 3950 50  0001 C CNN
+F 1 "+3.3V" H 1815 4273 50  0000 C CNN
+F 2 "" H 1800 4100 50  0001 C CNN
+F 3 "" H 1800 4100 50  0001 C CNN
+	1    1800 4100
+	1    0    0    -1
+$EndComp
+Wire Wire Line
+	1300 4900 1250 4900
+Wire Wire Line
+	1250 4900 1250 4100
+Wire Wire Line
+	1250 4100 1600 4100
+Connection ~ 1600 4100
+Wire Wire Line
+	1300 4700 1150 4700
+Wire Wire Line
+	1150 4700 1150 4650
+Wire Wire Line
+	1150 4650 1050 4650
+Wire Wire Line
+	1050 4550 1150 4550
+Wire Wire Line
+	1150 4550 1150 4500
+Wire Wire Line
+	1150 4500 1300 4500
+Wire Wire Line
+	10250 3800 10100 3800
+Wire Wire Line
+	10100 3800 10100 4900
+Connection ~ 10100 4900
+Wire Wire Line
+	10100 4900 10250 4900
+Wire Wire Line
+	5900 3950 5900 4250
+Wire Wire Line
+	5900 4250 6500 4250
+Connection ~ 6500 4250
+Wire Wire Line
+	1400 1000 2000 1000
+Connection ~ 1650 1200
+$Comp
 L power:GNDD #PWR0120
 U 1 1 5E6CE72E
@@
 $EndComp
 $Comp
-L Logic_LevelTranslator:TXS0102DCT U4
-U 1 1 5E6CF7FC
-P 1700 4600
-F 0 "U4" H 1700 4011 50  0000 C CNN
-F 1 "TXS0102DCT" H 1700 3920 50  0000 C CNN
-F 2 "Package_SO:SSOP-8_2.95x2.8mm_P0.65mm" H 1700 4050 50  0001 C CNN
-F 3 "http://www.ti.com/lit/gpn/txs0102" H 1700 4580 50  0001 C CNN
-	1    1700 4600
-	1    0    0    -1
-$EndComp
-$Comp
-L power:GNDD #PWR0121
-U 1 1 5E7470E9
-P 1700 5100
-F 0 "#PWR0121" H 1700 4850 50  0001 C CNN
-F 1 "GNDD" H 1704 4945 50  0000 C CNN
-F 2 "" H 1700 5100 50  0001 C CNN
-F 3 "" H 1700 5100 50  0001 C CNN
-	1    1700 5100
-	1    0    0    -1
-$EndComp
-$Comp
-L power:+5V #PWR0122
-U 1 1 5E74AF37
-P 1600 4100
-F 0 "#PWR0122" H 1600 3950 50  0001 C CNN
-F 1 "+5V" H 1615 4273 50  0000 C CNN
-F 2 "" H 1600 4100 50  0001 C CNN
-F 3 "" H 1600 4100 50  0001 C CNN
-	1    1600 4100
-	1    0    0    -1
-$EndComp
-$Comp
-L power:+3.3V #PWR0123
-U 1 1 5E74C9C1
-P 1800 4100
-F 0 "#PWR0123" H 1800 3950 50  0001 C CNN
-F 1 "+3.3V" H 1815 4273 50  0000 C CNN
-F 2 "" H 1800 4100 50  0001 C CNN
-F 3 "" H 1800 4100 50  0001 C CNN
-	1    1800 4100
-	1    0    0    -1
-$EndComp
-Wire Wire Line
-	1300 4900 1250 4900
-Wire Wire Line
-	1250 4900 1250 4100
-Wire Wire Line
-	1250 4100 1600 4100
-Connection ~ 1600 4100
-Wire Wire Line
-	1300 4700 1150 4700
-Wire Wire Line
-	1150 4700 1150 4650
-Wire Wire Line
-	1150 4650 1050 4650
-Wire Wire Line
-	1050 4550 1150 4550
-Wire Wire Line
-	1150 4550 1150 4500
-Wire Wire Line
-	1150 4500 1300 4500
-Wire Wire Line
-	10250 3800 10100 3800
-Wire Wire Line
-	10100 3800 10100 4900
-Connection ~ 10100 4900
-Wire Wire Line
-	10100 4900 10250 4900
+L power:+5V #PWR?
+U 1 1 5E5CCF95
+P 5900 950
+F 0 "#PWR?" H 5900 800 50  0001 C CNN
+F 1 "+5V" H 5915 1123 50  0000 C CNN
+F 2 "" H 5900 950 50  0001 C CNN
+F 3 "" H 5900 950 50  0001 C CNN
+	1    5900 950
+	1    0    0    -1
+$EndComp
 $EndSCHEMATC

Commit message: v0.0.9 pcb v1.0.2 changed USE_TFT_RESET in main.cpp
Parts:
- removed JP2: Backlight, Connector_PinHeader_2.54mm:PinHeader_1x03_P2.54mm_Vertical, symbol Jumper:Jumper_3_Open
- removed Q5: BC328, Package_TO_SOT_THT:TO-92_Inline, symbol Transistor_BJT:BC328
- removed R11: R, Resistor_THT:R_Axial_DIN0204_L3.6mm_D1.6mm_P7.62mm_Horizontal, symbol Device:R
- removed TR1: Backlight, Potentiometer_THT:Potentiometer_Piher_PT-10-V10_Vertical, symbol Device:R_POT_TRIM
- added unit 6 of U2
- U2: footprint Package_DIP:DIP-16_W7.62mm -> (none)
Connections:
- net +3V3: no longer J2.6 (Pin_6), J3.2 (Pin_2), U2.1 (VCC)
- net BL: now also U2.14
- net at J2.7 (Pin_7), J3.8 (Pin_8): now also U2.15
- new net: J2.6 (Pin_6), J3.2 (Pin_2), U2.1 (VCC)
Changed lines of the file:
@@
 F 0 "U2" H 10680 5496 50  0000 L CNN
 F 1 "4050" H 10680 5405 50  0000 L CNN
-F 2 "Package_DIP:DIP-16_W7.62mm" H 10450 5450 50  0001 C CNN
+F 2 "" H 10450 5450 50  0001 C CNN
 F 3 "http://www.intersil.com/content/dam/intersil/documents/cd40/cd4050bms.pdf" H 10450 5450 50  0001 C CNN
 	7    10450 5450
@@
 F 0 "U2" H 9100 5767 50  0000 C CNN
 F 1 "4050" H 9100 5676 50  0000 C CNN
-F 2 "Package_DIP:DIP-16_W7.62mm" H 9100 5450 50  0001 C CNN
+F 2 "" H 9100 5450 50  0001 C CNN
 F 3 "http://www.intersil.com/content/dam/intersil/documents/cd40/cd4050bms.pdf" H 9100 5450 50  0001 C CNN
 	5    9100 5450
@@
 F 0 "U2" H 9100 5417 50  0000 C CNN
 F 1 "4050" H 9100 5326 50  0000 C CNN
-F 2 "Package_DIP:DIP-16_W7.62mm" H 9100 5100 50  0001 C CNN
+F 2 "" H 9100 5100 50  0001 C CNN
 F 3 "http://www.intersil.com/content/dam/intersil/documents/cd40/cd4050bms.pdf" H 9100 5100 50  0001 C CNN
 	4    9100 5100
@@
 F 0 "U2" H 9100 5067 50  0000 C CNN
 F 1 "4050" H 9100 4976 50  0000 C CNN
-F 2 "Package_DIP:DIP-16_W7.62mm" H 9100 4750 50  0001 C CNN
+F 2 "" H 9100 4750 50  0001 C CNN
 F 3 "http://www.intersil.com/content/dam/intersil/documents/cd40/cd4050bms.pdf" H 9100 4750 50  0001 C CNN
 	3    9100 4750
@@
 F 0 "U2" H 9100 4717 50  0000 C CNN
 F 1 "4050" H 9100 4626 50  0000 C CNN
-F 2 "Package_DIP:DIP-16_W7.62mm" H 9100 4400 50  0001 C CNN
+F 2 "" H 9100 4400 50  0001 C CNN
 F 3 "http://www.intersil.com/content/dam/intersil/documents/cd40/cd4050bms.pdf" H 9100 4400 50  0001 C CNN
 	2    9100 4400
@@
 Wire Wire Line
 	9750 1950 9750 2100
-Text GLabel 9600 2450 0    50   Input ~ 0
-Tip
 Text GLabel 6500 3250 2    50   Input ~ 0
 Tip
@@
 	1    0    0    -1
 $EndComp
-$Comp
-L power:+3.3V #PWR0110
-U 1 1 5E8C1B71
-P 9200 3000
-F 0 "#PWR0110" H 9200 2850 50  0001 C CNN
-F 1 "+3.3V" H 9200 3150 50  0000 C CNN
-F 2 "" H 9200 3000 50  0001 C CNN
-F 3 "" H 9200 3000 50  0001 C CNN
-	1    9200 3000
-	1    0    0    -1
-$EndComp
 Wire Wire Line
 	10950 5450 10950 3900
@@
 F 0 "U2" H 9100 4367 50  0000 C CNN
 F 1 "4050" H 9100 4276 50  0000 C CNN
-F 2 "Package_DIP:DIP-16_W7.62mm" H 9100 4050 50  0001 C CNN
+F 2 "" H 9100 4050 50  0001 C CNN
 F 3 "http://www.intersil.com/content/dam/intersil/documents/cd40/cd4050bms.pdf" H 9100 4050 50  0001 C CNN
 	1    9100 4050
@@
 Wire Wire Line
 	10250 3700 10200 3700
-Connection ~ 10200 3700
 Wire Wire Line
 	10250 3600 9950 3600
@@
 Connection ~ 9950 3900
 Connection ~ 9950 3600
-$Comp
-L Transistor_BJT:BC328 Q5
-U 1 1 5E5AEB57
-P 9100 3250
-F 0 "Q5" H 9291 3296 50  0000 L CNN
-F 1 "BC328" H 9291 3205 50  0000 L CNN
-F 2 "Package_TO_SOT_THT:TO-92_Inline" H 9300 3175 50  0001 L CIN
-F 3 "http://www.redrok.com/PNP_BC327_-45V_-800mA_0.625W_Hfe100_TO-92.pdf" H 9100 3250 50  0001 L CNN
-	1    9100 3250
-	1    0    0    -1
-$EndComp
-Wire Wire Line
-	9950 3050 9200 3050
-Wire Wire Line
-	9200 3000 9200 3050
-Connection ~ 9200 3050
-Wire Wire Line
-	9200 3700 9200 3450
-Wire Wire Line
-	9200 3700 10200 3700
-$Comp
-L Device:R R11
-U 1 1 5E5DD438
-P 8750 3250
-F 0 "R11" V 8543 3250 50  0000 C CNN
-F 1 "R" V 8634 3250 50  0000 C CNN
-F 2 "Resistor_THT:R_Axial_DIN0204_L3.6mm_D1.6mm_P7.62mm_Horizontal" V 8680 3250 50  0001 C CNN
-F 3 "~" H 8750 3250 50  0001 C CNN
-	1    8750 3250
-	0    1    1    0
-$EndComp
-$Comp
-L Device:R_POT_TRIM TR1
-U 1 1 5E5DED2E
-P 8450 2850
-F 0 "TR1" V 8243 2850 50  0000 C CNN
-F 1 "Backlight" V 8334 2850 50  0000 C CNN
-F 2 "Potentiometer_THT:Potentiometer_Piher_PT-10-V10_Vertical" H 8450 2850 50  0001 C CNN
-F 3 "~" H 8450 2850 50  0001 C CNN
-	1    8450 2850
-	0    1    1    0
-$EndComp
-$Comp
-L Jumper:Jumper_3_Open JP2
-U 1 1 5E5E0E31
-P 8450 3250
-F 0 "JP2" V 8496 3337 50  0000 L CNN
-F 1 "Backlight" V 8405 3337 50  0000 L CNN
-F 2 "Connector_PinHeader_2.54mm:PinHeader_1x03_P2.54mm_Vertical" H 8450 3250 50  0001 C CNN
-F 3 "~" H 8450 3250 50  0001 C CNN
-	1    8450 3250
-	0    -1   -1   0
-$EndComp
-Text GLabel 8450 3500 3    50   Input ~ 0
+Text GLabel 8800 3700 0    50   Input ~ 0
 BL
 Text GLabel 6500 3550 2    50   Input ~ 0
 BL
-Wire Wire Line
-	8600 2850 8950 2850
-Wire Wire Line
-	8950 2850 8950 3050
-Wire Wire Line
-	8950 3050 9200 3050
-Wire Wire Line
-	8300 2850 8100 2850
-Wire Wire Line
-	8100 2850 8100 2900
 $Comp
 L Logic_LevelTranslator:TXS0102DCT U4
@@
 Wire Wire Line
 	1400 1000 2000 1000
-Connection ~ 1650 1200
-$Comp
-L power:GNDD #PWR0120
-U 1 1 5E6CE72E
-P 8100 2900
-F 0 "#PWR0120" H 8100 2650 50  0001 C CNN
-F 1 "GNDD" H 8104 2745 50  0000 C CNN
-F 2 "" H 8100 2900 50  0001 C CNN
-F 3 "" H 8100 2900 50  0001 C CNN
-	1    8100 2900
-	1    0    0    -1
-$EndComp
 $Comp
 L power:+5V #PWR?
@@
 	1    0    0    -1
 $EndComp
+$Comp
+L 4xxx:4050 U2
+U 6 1 5E57BA7A
+P 9100 3700
+F 0 "U2" H 9100 4017 50  0000 C CNN
+F 1 "4050" H 9100 3926 50  0000 C CNN
+F 2 "" H 9100 3700 50  0001 C CNN
+F 3 "http://www.intersil.com/content/dam/intersil/documents/cd40/cd4050bms.pdf" H 9100 3700 50  0001 C CNN
+	6    9100 3700
+	1    0    0    -1
+$EndComp
+Text GLabel 9600 2450 0    50   Input ~ 0
+Tip
+Wire Wire Line
+	9400 3700 10200 3700
+Connection ~ 10200 3700
 $EndSCHEMATC

Commit message: v0.0.10
Parts:
- removed J8: I2C, Connector_PinHeader_2.54mm:PinHeader_1x04_P2.54mm_Vertical, symbol Connector:Conn_01x04_Female
- removed JP1: USE_TFT_RESET, Connector_PinHeader_2.54mm:PinHeader_1x03_P2.54mm_Vertical, symbol Device:Jumper_NC_Dual
- added C3, C4, C5: 100nF, Capacitor_THT:C_Disc_D4.3mm_W1.9mm_P5.00mm, symbol Device:C
- added J8: I2C, Connector_PinHeader_2.54mm:PinHeader_1x04_P2.54mm_Vertical, symbol Connector:Conn_01x04_Male
- added JP1: TFT Reset, Connector_PinHeader_2.54mm:PinHeader_1x03_P2.54mm_Vertical, symbol Jumper:Jumper_3_Bridged12
- added JP2: BL Control, Connector_PinHeader_2.54mm:PinHeader_1x03_P2.54mm_Vertical, symbol Jumper:Jumper_3_Bridged12
- added R9: 10kΩ, Resistor_THT:R_Axial_DIN0204_L3.6mm_D1.6mm_P7.62mm_Horizontal, symbol Device:R
- U2: footprint (none) -> Package_DIP:DIP-16_W7.62mm
- U4: footprint Package_SO:SSOP-8_2.95x2.8mm_P0.65mm -> Package_DIP:DIP-8_W7.62mm
Connections:
- net +5V: now also J2.6 (Pin_6), J3.2 (Pin_2), U1.20 (AVCC), U2.1 (VCC), C3.1, C4.1, C5.2, J8.1 (Pin_1), R9.1
- net BL: now also JP2.1 (A); no longer U2.14
- net GNDD: now also C3.2, C4.2, C5.1, J8.4 (Pin_4)
- net Res: now also JP1.1 (A)
- net TFT-RST: now also JP1.3 (B)
- net at U2.7: now also JP1.2 (C)
- net at U4.5 (A1): now also J8.2 (Pin_2)
- net at U4.4 (A2): now also J8.3 (Pin_3)
- net +12C renamed +12V
- net T+ renamed Up
- net T- renamed Down
- new net: JP2.2 (C), U2.14
- new net: JP2.3 (B), R9.2
- no-connect marks 0 -> 32
Other:
- note added: "Heat/temperatur control"
- note added: "ISP / I2C"
- note added: "Input"
- note added: "Power supply"
- note added: "TFT control"
