File: pcb/circuit.sch (KiCad schematic (older format))
At the start: 48 parts, among them IC1 OP703PA, J1 Soldering iron, J2 TFT AK, J3 TFT RL, J4 12V, J5 Power 12V, J6 LiPo-Bal, J8 I2C, J9 ISP, Q1 IRF5305, Q2 2N7000, Q3 LM7805, Q4 LM117T 3.3, SW1 T1, SW2 T2, SW3 T3, SW7 Menu, U1 ATmega328-PU, U2 4050, U3 LM4040LP-4.1, U4 TXS0102DCT, Y1 16MHz

Commit message: v0.0.11
Parts:
- J1: footprint Connector_Phoenix_MSTB:PhoenixContact_MSTBVA_2,5_4-G_1x04_P5.00mm_Vertical -> TerminalBlock_Phoenix:TerminalBlock_Phoenix_MKDS-1,5-4-5.08_1x04_P5.08mm_Horizontal
- J5: footprint Connector_Phoenix_MSTB:PhoenixContact_MSTBVA_2,5_2-G-5,08_1x02_P5.08mm_Vertical -> TerminalBlock_Phoenix:TerminalBlock_Phoenix_MKDS-1,5-2-5.08_1x02_P5.08mm_Horizontal
- Q1, Q3, Q4: footprint Package_TO_SOT_THT:TO-220-3_Vertical -> Package_TO_SOT_THT:TO-220-3_Horizontal_TabDown
- Y1: footprint Crystal:Crystal_HC18-U_Vertical -> Crystal:Crystal_HC49-U_Vertical
Connections:
- net VMEM is gone; now on net AREF: U1.21 (AREF)
- net +12V: no longer R20.1
- net +5V: now also R20.2
- net AREF: now reaches U3.2 (K)
- net AREF: now also R20.1; no longer R20.2
Changed lines of the file:
@@
 Title "soldering station"
 Date "2020-02-28"
-Rev "1.0.0"
-Comp "KARL"
+Rev "1.0.1"
+Comp "(c) by KARL"
 Comment1 ""
 Comment2 ""
@@
 F 0 "Q1" V 10543 1350 50  0000 C CNN
 F 1 "IRF5305" V 10452 1350 50  0000 C CNN
-F 2 "Package_TO_SOT_THT:TO-220-3_Vertical" H 10400 1275 50  0001 L CIN
+F 2 "Package_TO_SOT_THT:TO-220-3_Horizontal_TabDown" H 10400 1275 50  0001 L CIN
 F 3 "http://www.infineon.com/dgdl/irf4905.pdf?fileId=5546d462533600a4015355e32165197c" H 10200 1350 50  0001 L CNN
 	1    10200 1350
@@
 F 0 "J1" H 10487 1642 50  0000 L CNN
 F 1 "Soldering iron" H 107730 1551 50  0000 L CNN
-F 2 "Connector_Phoenix_MSTB:PhoenixContact_MSTBVA_2,5_4-G_1x04_P5.00mm_Vertical" H 10800 1650 50  0001 C CNN
+F 2 "TerminalBlock_Phoenix:TerminalBlock_Phoenix_MKDS-1,5-4-5.08_1x04_P5.08mm_Horizontal" H 10800 1650 50  0001 C CNN
 F 3 "~" H 10800 1650 50  0001 C CNN
 	1    10800 1650
@@
 L power:+3V3 #PWR0105
 U 1 1 5E605821
-P 2600 1600
-F 0 "#PWR0105" H 2600 1450 50  0001 C CNN
-F 1 "+3V3" H 2615 1773 50  0000 C CNN
-F 2 "" H 2600 1600 50  0001 C CNN
-F 3 "" H 2600 1600 50  0001 C CNN
-	1    2600 1600
+P 2800 1600
+F 0 "#PWR0105" H 2800 1450 50  0001 C CNN
+F 1 "+3V3" H 2815 1773 50  0000 C CNN
+F 2 "" H 2800 1600 50  0001 C CNN
+F 3 "" H 2800 1600 50  0001 C CNN
+	1    2800 1600
 	-1   0    0    -1
-$EndComp
-$Comp
-L power:+5V #PWR0106
-U 1 1 5E6063C7
-P 2600 1000
-F 0 "#PWR0106" H 2600 850 50  0001 C CNN
-F 1 "+5V" H 2615 1173 50  0000 C CNN
-F 2 "" H 2600 1000 50  0001 C CNN
-F 3 "" H 2600 1000 50  0001 C CNN
-	1    2600 1000
-	1    0    0    -1
 $EndComp
 $Comp
@@
 U 1 1 5E6832F5
 P 5550 1900
-F 0 "Y1" H 5550 2168 50  0000 C CNN
+F 0 "Y1" V 5550 1900 50  0000 C CNN
 F 1 "16MHz" H 5850 1900 50  0000 C CNN
-F 2 "Crystal:Crystal_HC18-U_Vertical" H 5550 1900 50  0001 C CNN
+F 2 "Crystal:Crystal_HC49-U_Vertical" H 5550 1900 50  0001 C CNN
 F 3 "~" H 5550 1900 50  0001 C CNN
 	1    5550 1900
@@
 T2
 Text GLabel 1250 6900 2    50   Input ~ 0
-MISO
+T3
 Text GLabel 2350 6900 2    50   Input ~ 0
 Up
@@
 $EndComp
 Wire Wire Line
-	1650 1000 1650 1200
-Wire Wire Line
-	2000 1000 2000 1200
-Wire Wire Line
-	2000 1200 2000 1500
-Connection ~ 2000 1200
-Wire Wire Line
-	2000 1500 2000 1600
-Connection ~ 2000 1500
-Connection ~ 1400 1200
-Wire Wire Line
-	1150 1500 2000 1500
-$Comp
-L power:VMEM #PWR0108
-U 1 1 5E67A481
-P 1650 1000
-F 0 "#PWR0108" H 1650 850 50  0001 C CNN
-F 1 "VMEM" H 1665 1173 50  0000 C CNN
-F 2 "" H 1650 1000 50  0001 C CNN
-F 3 "" H 1650 1000 50  0001 C CNN
-	1    1650 1000
-	-1   0    0    -1
-$EndComp
-Wire Wire Line
-	1400 1300 2300 1300
-Wire Wire Line
 	1150 1600 1250 1600
-Connection ~ 1400 1300
-Wire Wire Line
-	1400 1200 1400 1300
-Connection ~ 2000 1000
+Connection ~ 2100 1000
 Connection ~ 1400 1600
 $Comp
@@
 	1    0    0    -1
 $EndComp
-Wire Wire Line
-	1400 1600 1400 1300
-Connection ~ 2300 1300
 $Comp
 L Regulator_Linear:LM7805_TO220 Q4
 U 1 1 5E601A73
-P 2300 1600
-F 0 "Q4" H 2300 1842 50  0000 C CNN
-F 1 "LM117T 3.3" H 2300 1751 50  0000 C CNN
-F 2 "Package_TO_SOT_THT:TO-220-3_Vertical" H 2300 1825 50  0001 C CIN
-F 3 "http://www.fairchildsemi.com/ds/LM/LM7805.pdf" H 2300 1550 50  0001 C CNN
-	1    2300 1600
+P 2400 1600
+F 0 "Q4" H 2400 1842 50  0000 C CNN
+F 1 "LM117T 3.3" H 2400 1751 50  0000 C CNN
+F 2 "Package_TO_SOT_THT:TO-220-3_Horizontal_TabDown" H 2400 1825 50  0001 C CIN
+F 3 "http://www.fairchildsemi.com/ds/LM/LM7805.pdf" H 2400 1550 50  0001 C CNN
+	1    2400 1600
 	1    0    0    1
 $EndComp
@@
 L Regulator_Linear:LM7805_TO220 Q3
 U 1 1 5E5FF5BA
-P 2300 1000
-F 0 "Q3" H 2300 1242 50  0000 C CNN
-F 1 "LM7805" H 2300 1151 50  0000 C CNN
-F 2 "Package_TO_SOT_THT:TO-220-3_Vertical" H 2300 1225 50  0001 C CIN
-F 3 "http://www.fairchildsemi.com/ds/LM/LM7805.pdf" H 2300 950 50  0001 C CNN
-	1    2300 1000
+P 2400 1000
+F 0 "Q3" H 2400 1242 50  0000 C CNN
+F 1 "LM7805" H 2400 1151 50  0000 C CNN
+F 2 "Package_TO_SOT_THT:TO-220-3_Horizontal_TabDown" H 2400 1225 50  0001 C CIN
+F 3 "http://www.fairchildsemi.com/ds/LM/LM7805.pdf" H 2400 950 50  0001 C CNN
+	1    2400 1000
 	1    0    0    -1
 $EndComp
@@
 F 0 "J5" H 868 1717 50  0000 C CNN
 F 1 "Power 12V" H 868 1626 50  0000 C CNN
-F 2 "Connector_Phoenix_MSTB:PhoenixContact_MSTBVA_2,5_2-G-5,08_1x02_P5.08mm_Vertical" H 950 1500 50  0001 C CNN
+F 2 "TerminalBlock_Phoenix:TerminalBlock_Phoenix_MKDS-1,5-2-5.08_1x02_P5.08mm_Horizontal" H 950 1500 50  0001 C CNN
 F 3 "~" H 950 1500 50  0001 C CNN
 	1    950  1500
 	-1   0    0    -1
-$EndComp
-$Comp
-L Device:R R20
-U 1 1 5E509E69
-P 1850 1200
-F 0 "R20" H 1920 1246 50  0000 L CNN
-F 1 "560Ω" H 1920 1155 50  0000 L CNN
-F 2 "Resistor_THT:R_Axial_DIN0204_L3.6mm_D1.6mm_P7.62mm_Horizontal" V 1780 1200 50  0001 C CNN
-F 3 "~" H 1850 1200 50  0001 C CNN
-	1    1850 1200
-	0    1    -1   0
 $EndComp
 Connection ~ 7400 1750
@@
 	1    0    0    -1
 $EndComp
-Text GLabel 5400 1600 2    50   Input ~ 0
+Text GLabel 5700 1550 2    50   Input ~ 0
 MISO
 Text GLabel 1100 3650 0    50   Input ~ 0
@@
 SCL
 $Comp
-L power:VMEM #PWR0111
-U 1 1 5E9EB7A8
-P 4200 1200
-F 0 "#PWR0111" H 4200 1050 50  0001 C CNN
-F 1 "VMEM" V 4215 1328 50  0000 L CNN
-F 2 "" H 4200 1200 50  0001 C CNN
-F 3 "" H 4200 1200 50  0001 C CNN
-	1    4200 1200
-	0    -1   -1   0
-$EndComp
-$Comp
 L MCU_Microchip_ATmega:ATmega328-PU U1
 U 1 1 5E4F8E4A
@@
 	4800 4200 5400 4200
 Connection ~ 5400 4200
-Wire Wire Line
-	1400 1000 2000 1000
 $Comp
 L power:+5V #PWR0110
@@
 L power:+12V #PWR0120
 U 1 1 5E5B0C7D
-P 2000 1000
-F 0 "#PWR0120" H 2000 850 50  0001 C CNN
-F 1 "+12V" H 2015 1173 50  0000 C CNN
-F 2 "" H 2000 1000 50  0001 C CNN
-F 3 "" H 2000 1000 50  0001 C CNN
-	1    2000 1000
+P 2100 1000
+F 0 "#PWR0120" H 2100 850 50  0001 C CNN
+F 1 "+12V" H 2115 1173 50  0000 C CNN
+F 2 "" H 2100 1000 50  0001 C CNN
+F 3 "" H 2100 1000 50  0001 C CNN
+	1    2100 1000
 	1    0    0    -1
 $EndComp
@@
 Wire Notes Line
 	750  3150 750  650
-Wire Notes Line
-	750  650  2800 650
-Wire Notes Line
-	2800 650  2800 3150
-Wire Notes Line
-	2800 3150 750  3150
+Text GLabel 5700 1650 2    50   Input ~ 0
+T3
+Wire Wire Line
+	5700 1550 5650 1550
+Wire Wire Line
+	5650 1550 5650 1600
+Wire Wire Line
+	5650 1650 5700 1650
+Wire Wire Line
+	5400 1600 5650 1600
+Connection ~ 5650 1600
+Wire Wire Line
+	5650 1600 5650 1650
+Text GLabel 4200 1200 0    50   Output ~ 0
+AREF
+Text GLabel 1750 950  1    50   Input ~ 0
+AREF
+Wire Wire Line
+	4250 1200 4200 1200
+Wire Wire Line
+	1400 1200 1400 1300
+Connection ~ 1400 1200
+Connection ~ 2100 1500
+Wire Wire Line
+	2100 1500 2100 1600
+Wire Wire Line
+	1700 1200 1750 1200
+Wire Wire Line
+	1400 1000 2100 1000
+Wire Wire Line
+	1750 950  1750 1200
+Connection ~ 1750 1200
+Wire Wire Line
+	1750 1200 1800 1200
+Connection ~ 2400 1300
+Connection ~ 1400 1300
+Wire Wire Line
+	1400 1300 1400 1600
+Wire Notes Line
+	750  650  2950 650
+Wire Notes Line
+	2950 650  2950 3150
+Wire Notes Line
+	2950 3150 750  3150
+$Comp
+L power:+5V #PWR0106
+U 1 1 5E6063C7
+P 2800 1000
+F 0 "#PWR0106" H 2800 850 50  0001 C CNN
+F 1 "+5V" H 2800 1200 50  0000 C CNN
+F 2 "" H 2800 1000 50  0001 C CNN
+F 3 "" H 2800 1000 50  0001 C CNN
+	1    2800 1000
+	1    0    0    -1
+$EndComp
+Wire Wire Line
+	2700 1000 2800 1000
+Wire Wire Line
+	2800 1600 2700 1600
+Wire Wire Line
+	2100 1000 2100 1500
+Wire Wire Line
+	2400 1300 1400 1300
+$Comp
+L Device:R R20
+U 1 1 5E509E69
+P 1800 1350
+F 0 "R20" H 1870 1396 50  0000 L CNN
+F 1 "560Ω" H 1870 1305 50  0000 L CNN
+F 2 "Resistor_THT:R_Axial_DIN0204_L3.6mm_D1.6mm_P7.62mm_Horizontal" V 1730 1350 50  0001 C CNN
+F 3 "~" H 1800 1350 50  0001 C CNN
+	1    1800 1350
+	-1   0    0    -1
+$EndComp
+Wire Wire Line
+	1800 1500 1800 1900
+Wire Wire Line
+	1800 1900 2900 1900
+Wire Wire Line
+	2900 1900 2900 1000
+Wire Wire Line
+	2900 1000 2800 1000
+Connection ~ 2800 1000
+Wire Wire Line
+	1150 1500 2100 1500
 $EndSCHEMATC
