File: KiCad/circuit.kicad_pcb (KiCad board)
At the start: 2 copper layers, 100 x 100 mm, 47 parts, among them IC1 OP703PA, J1 Soldering iron, J2 TFT AK, J3 TFT RL, J4 12V, J5 Power 12V, J6 LiPo-Bal, J8 I2C, J9 ISP, Q1 IRF5305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

Commit message: v0.0.12
Parts:
- added 10x24: Proto10x24, my:Proto10x24, F.Cu at (84.5, 56.8)
- added 1x24: Proto1x24, my:Proto1x24, F.Cu at (57.8, 59.3)
- added A1: Arduino_Nano_v3.x, Module:Arduino_Nano, F.Cu at (146.1, 48.0)
- added C6: 100nf, Capacitor_THT:C_Disc_D4.3mm_W1.9mm_P5.00mm, F.Cu at (36.4, 93.3)
- added C7: 100nF, Capacitor_THT:C_Disc_D4.3mm_W1.9mm_P5.00mm, F.Cu at (31.4, 108.6)
- added Neo-5V: PinHeader_1x01_P2.54mm_Vertical, Connector_PinHeader_2.54mm:PinHeader_1x01_P2.54mm_Vertical, F.Cu at (106.6, 70.0)
- added PB0-GND: PinHeader_1x01_P2.54mm_Vertical, Connector_PinHeader_2.54mm:PinHeader_1x01_P2.54mm_Vertical, F.Cu at (92.3, 109.8)
- added PD6-GND: PinHeader_1x01_P2.54mm_Vertical, Connector_PinHeader_2.54mm:PinHeader_1x01_P2.54mm_Vertical, F.Cu at (92.4, 114.9)
- J6: footprint Connector_JST:JST_EH_B4B-EH-A_1x04_P2.50mm_Vertical -> Connector_JST:JST_EH_S4B-EH_1x04_P2.50mm_Horizontal
- J8, J9: moved to B.Cu
- moved C4 99.9 mm to (38.0, 54.5), turned to 90 degrees
- moved C5 49.4 mm to (82.4, 81.1), turned to 90 degrees
- moved C3 41.5 mm to (68.2, 103.3)
- moved R20 35.5 mm to (38.5, 42.3), turned to 0 degrees
- moved R9 29.4 mm to (105.5, 107.3), turned to 270 degrees
- moved R24 27.1 mm to (40.6, 75.5), turned to 180 degrees
- moved U2 17.9 mm to (79.4, 75.2), turned to 270 degrees
- moved JP1 12.1 mm to (95.2, 109.8), turned to 90 degrees
- moved R8 10.9 mm to (116.2, 34.7)
- moved R4 10.6 mm to (51.2, 59.9), turned to 180 degrees
- moved U3 10.3 mm to (34.9, 31.1), turned to 0 degrees
- moved JP2 9.55 mm to (95.2, 114.9), turned to 90 degrees
- moved R3 8.20 mm to (51.6, 49.4)
- moved C2 6.83 mm to (35.7, 70.5), turned to 0 degrees
- moved C1 6.47 mm to (50.5, 47.0), turned to 90 degrees
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Connections:
- C5 pad 2: +5V -> +3V3
- J2 pad 6: +5V -> +3V3
- J3 pad 2: +5V -> +3V3
- JP1 pad 1: Res -> TFT-RST
- JP1 pad 3: TFT-RST -> Res
- R20 pad 1: +12V -> AREF
- R20 pad 2: Net-(R20-Pad2) -> +5V
- U1 pad 21: VMEM -> AREF
- U2 pad 1: +5V -> +3V3
- U3 pad 2: Net-(R20-Pad2) -> AREF
Routing:
- net +5V: track 0.00 -> 64.3 mm
- net GNDD: track 212.8 -> 245.8 mm
- net Net-(C1-Pad1): track 0.04 -> 17.3 mm
- net Net-(J1-Pad2): track 0.80 -> 15.5 mm
- net BL: track 14.2 -> 0.00 mm
- net AREF: track 0.00 -> 13.2 mm
- net Net-(IC1-Pad2): track 0.00 -> 12.9 mm
- net Net-(Q2-Pad2): track 75.5 -> 82.0 mm
- net Sensor: track 0.00 -> 6.34 mm, vias 0 -> 1
- net Net-(IC1-Pad6): track 0.00 -> 5.77 mm
- net Net-(J6-Pad3): track 5.14 -> 0.00 mm
- net Net-(J6-Pad2): track 5.12 -> 0.00 mm
- net Net-(J6-Pad1): track 5.12 -> 0.00 mm
- net +12V: track 107.3 -> 105.4 mm
- net +3V3: track 0.00 -> 1.50 mm, vias 0 -> 1
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Other:
- board text added: "(c) by KARL"
- board text added: "HW Rev. 4.0"

Commit message: v0.0.13
Parts:
- removed A1: Arduino_Nano_v3.x, Module:Arduino_Nano
Routing:
- net GNDD: track 245.8 -> 507.3 mm
- net +3V3: track 1.50 -> 205.3 mm, vias 1 -> 0
- net +5V: track 64.3 -> 260.1 mm
- net Tip: track 0.00 -> 106.5 mm
- net Res: track 0.00 -> 95.4 mm
- net MISO: track 0.00 -> 85.1 mm
- net SCK: track 0.00 -> 82.2 mm, vias 0 -> 1
- net Net-(J2-Pad7): track 0.00 -> 73.9 mm
- net AREF: track 13.2 -> 80.2 mm
- net MOSI: track 0.00 -> 66.9 mm, vias 2 -> 1
- net Up: track 0.00 -> 65.4 mm
- net Net-(J2-Pad3): track 0.00 -> 62.0 mm
- net Pow: track 0.00 -> 61.3 mm
- net Net-(J2-Pad2): track 0.00 -> 60.9 mm
- net Net-(J2-Pad1): track 0.00 -> 60.8 mm
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Other:
- rule trace_min: 0.5 -> 0.25

Commit message: v1.0.1 / HW Rev. 4.0.1
Parts:
- removed 1x24: Proto1x24, my:Proto1x24
- removed J8: I2C, Connector_PinHeader_2.54mm:PinHeader_1x04_P2.54mm_Vertical
- removed Neo-5V, PB0-GND, PD6-GND: PinHeader_1x01_P2.54mm_Vertical, Connector_PinHeader_2.54mm:PinHeader_1x01_P2.54mm_Vertical
- added Logo1: LOGO, my:Logo, B.Cu at (30.5, 111.4)
- added Logo1: LOGO, my:Logo, F.Cu at (36.2, 111.4)
- added Prototype1: Conn_01x24, my:Proto1x24, F.Cu at (57.8, 59.3)
- D1: value LED -> NeoPixel_THT; footprint Diode_THT:D_DO-15_P2.54mm_Vertical_AnodeUp -> LED_THT:LED_D5.0mm-4_RGB
- moved C7 59.4 mm to (78.1, 71.9), turned to 270 degrees
- moved C6 57.9 mm to (92.0, 76.9), turned to 90 degrees
- moved U4 48.7 mm to (81.2, 78.1), turned to 90 degrees
- moved C5 32.6 mm to (51.0, 72.6), turned to 270 degrees
- moved U2 24.9 mm to (54.6, 78.2), turned to 90 degrees
- moved J3 4.46 mm to (43.6, 67.4)
- moved SW2 3.13 mm to (67.9, 109.1)
- moved SW3 3.13 mm to (53.7, 109.2)
- moved SW1 3.13 mm to (81.7, 109.2)
- moved D1 3.08 mm to (108.7, 70.8), turned to 0 degrees
- moved U1 1.62 mm to (54.4, 98.9)
- moved Y1 1.45 mm to (81.9, 103.8)
- moved C3 1.20 mm to (67.1, 102.7)
- moved R8 0.72 mm to (116.8, 35.1)
Connections:
- D1 pad 1: GNDD -> Net-(D1-Pad1)
- D1 pad 2: Net-(D1-Pad2) -> GNDD
- J1 pad 3: Net-(J1-Pad3) -> Tip2
- R10 pad 1: Net-(D1-Pad2) -> Net-(Prototype1-Pad11)
- R10 pad 2: Net-(R10-Pad2) -> Net-(D1-Pad4)
- U1 pad 13: Net-(R10-Pad2) -> Net-(Prototype1-Pad11)
- U4 pad 4: Net-(J8-Pad3) -> SCL5V
- U4 pad 5: Net-(J8-Pad2) -> SDA5V
Routing:
- net Tip2: track 0.00 -> 79.7 mm, vias 0 -> 1
- net Net-(Prototype1-Pad11): track 0.00 -> 78.2 mm
- net +5V: track 260.1 -> 336.5 mm
- net BL: track 20.3 -> 75.8 mm, vias 0 -> 1
- net SCL: track 20.9 -> 72.5 mm
- net TFT-RST: track 12.4 -> 60.8 mm
- net Sensor: track 39.8 -> 86.4 mm, vias 0 -> 1
- net Res: track 95.4 -> 139.1 mm
- net Net-(D1-Pad4): track 0.00 -> 43.2 mm
- net Net-(J2-Pad5): track 60.7 -> 99.6 mm
- net SCL5V: track 0.00 -> 34.6 mm
- net Tip: track 106.5 -> 139.0 mm
- net Net-(J2-Pad4): track 59.1 -> 91.0 mm
- net Net-(D1-Pad1): track 0.00 -> 30.5 mm
- net Net-(J2-Pad2): track 60.9 -> 91.2 mm
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Other:
- board text added: "(c) by KARL HW Rev. 4.0.1"
- board text removed: "(c) by KARL"
- board text removed: "HW Rev. 4.0"

Commit message: v1.0.1
Parts:
- moved Logo1 3.11 mm to (33.6, 111.4)
- moved Logo1 2.51 mm to (33.7, 111.3)
Routing:
- net +5V: track 336.5 -> 330.8 mm
Other:
- board text added: "JLCJLCJLCJLC"
Changed lines of the file:
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@@
   (general
     (thickness 1.6)
-    (drawings 10)
-    (tracks 753)
+    (drawings 11)
+    (tracks 750)
     (zones 0)
     (modules 52)
@@
     (visible_elements FEFDA66F)
     (pcbplotparams
-      (layerselection 0x010fc_ffffffff)
+      (layerselection 0x010f0_ffffffff)
       (usegerberextensions false)
       (usegerberattributes false)
@@
   )
   (module my:Logo locked (layer B.Cu)
-    (at 30.52572 111.38408 180)
+    (at 33.63468 111.37646 180)
     (fp_text reference Logo1 (at 0 0) (layer B.SilkS) hide
       (effects (font (size 1.524 1.524) (thickness 0.3)) (justify mirror))
@@
   )
   (module my:Logo locked (layer F.Cu)
-    (at 36.16706 111.38408)
+    (at 33.655 111.34852)
     (fp_text reference Logo1 (at 0 0) (layer F.SilkS) hide
       (effects (font (size 1.524 1.524) (thickness 0.3)))
@@
     )
   )
+  (gr_text JLCJLCJLCJLC (at 116.45646 104.2162 90) (layer B.SilkS)
+    (effects (font (size 1 1) (thickness 0.15)) (justify mirror))
+  )
   (gr_text "(c) by KARL\nHW Rev. 4.0.1" (at 25.23744 116.52504) (layer F.Cu)
     (effects (font (size 1.5 1.5) (thickness 0.3)) (justify left))
@@
   (segment (start 106.6685 106.1205) (end 105.474 107.315) (width 0.25) (layer B.Cu) (net 17))
   (segment (start 26.035 93.726) (end 27.3103 93.726) (width 0.25) (layer B.Cu) (net 17))
-  (segment (start 45.9875 61.1166) (end 42.2959 64.8082) (width 0.25) (layer B.Cu) (net 17))
-  (segment (start 42.2959 64.8082) (end 41.8008 64.8082) (width 0.25) (layer B.Cu) (net 17))
   (segment (start 45.9875 57.1365) (end 45.9875 61.1166) (width 0.25) (layer B.Cu) (net 17))
   (segment (start 45.9875 61.1166) (end 53.5321 61.1166) (width 0.25) (layer B.Cu) (net 17))
@@
   (segment (start 53.229 30.21) (end 68.2046 30.21) (width 1) (layer B.Cu) (net 17))
   (segment (start 46.101 37.338) (end 46.801 36.638) (width 1) (layer B.Cu) (net 17))
-  (segment (start 41.8007 64.8082) (end 41.8008 64.8082) (width 0.25) (layer B.Cu) (net 17))
   (segment (start 68.2046 30.21) (end 68.2046 30.1959) (width 1) (layer B.Cu) (net 17))
   (segment (start 46.801 36.638) (end 46.101 37.338) (width 1) (layer B.Cu) (net 17))
