File: KiCad/circuit.kicad_pcb (KiCad board)
At the start: 2 copper layers, 100 x 100 mm, 52 parts, among them IC1 OP703PA, J1 Soldering iron, J2 TFT AK, J3 TFT RL, J4 12V, J5 Power 12V, J6 LiPo-Bal, J9 ISP, Q1 IRF5305, Q2 2N7000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

Commit message: v1.0.5 minor changes in schematic and pcb
Parts:
- J1, J5: moved to B.Cu
- R10: value R -> 220Ω/0Ω
